File: Layout/Console Interface/Wireless.kicad_sch (KiCad schematic)
At the start: 5 parts

Commit message: Use separate board for lights
Parts:
- D8, D9: footprint LED_SMD:LED_0805_2012Metric -> LED_SMD:LED_0603_1608Metric
- R16, R17: footprint Resistor_SMD:R_0805_2012Metric -> Resistor_SMD:R_0603_1608Metric
Changed lines of the file:
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@@
       (effects (font (size 1.27 1.27)) (justify right))
     )
-    (property "Footprint" "LED_SMD:LED_0805_2012Metric" (at 186.436 88.011 0)
+    (property "Footprint" "LED_SMD:LED_0603_1608Metric" (at 186.436 88.011 0)
       (effects (font (size 1.27 1.27)) hide)
     )
@@
       (effects (font (size 1.27 1.27)) (justify left))
     )
-    (property "Footprint" "Resistor_SMD:R_0805_2012Metric" (at 174.752 80.645 90)
+    (property "Footprint" "Resistor_SMD:R_0603_1608Metric" (at 174.752 80.645 90)
       (effects (font (size 1.27 1.27)) hide)
     )
@@
       (effects (font (size 1.27 1.27)) (justify right))
     )
-    (property "Footprint" "LED_SMD:LED_0805_2012Metric" (at 173.736 88.011 0)
+    (property "Footprint" "LED_SMD:LED_0603_1608Metric" (at 173.736 88.011 0)
       (effects (font (size 1.27 1.27)) hide)
     )
@@
       (effects (font (size 1.27 1.27)) (justify left))
     )
-    (property "Footprint" "Resistor_SMD:R_0805_2012Metric" (at 187.452 80.645 90)
-      (effects (font (size 1.27 1.27)) hide)
-    )
+    (property "Footprint" "Resistor_SMD:R_0603_1608Metric" (at 187.452 80.645 90)
+      (effects (font (size 1.27 1.27)) hide)
+    )
