File: Layout/Controller Interface/processor.kicad_sch (KiCad schematic)
At the start: 26 parts, among them J1 USB_C_Receptacle_USB2.0, J5 Conn_01x08_Socket, SW3 SW_PAIR, SW4 SW_BOOT, U1 W25Q32JVSS, U2 RP2040, Y2 Crystal_GND24

Commit message: Update KiCAD project
Parts:
- added J8: Conn_01x03_Pin, Connector_PinHeader_2.54mm:PinHeader_1x03_P2.54mm_Vertical, symbol Connector:Conn_01x03_Pin
Connections:
- net GND: now also J8.3 (Pin_3)
- net SWCLK: now reaches U2.24 (SWCLK)
- net SWCLK: now also J8.2 (Pin_2)
- net SWD: now reaches U2.25 (SWD)
- net SWD: now also J8.1 (Pin_1)
